File: cncpatch/cncpatch.kicad_pcb (KiCad board)
At the start: 2 copper layers, 36 x 72 mm, 40 parts, among them J1 Conn_01x03_Socket, J2 Conn_01x03_Socket, J3 Conn_01x03_Socket, J4 Conn_01x03_Socket, J5 Conn_01x03_Socket, J6 Conn_01x03_Socket, J7 Conn_01x08_Socket, Q1 BC858, Q2 BC858, Q3 BC858, Q4 AO3401A, U2 PC817

Commit message: Typos and reord
Parts:
- removed Q1, Q2, Q3: BC858, Package_TO_SOT_SMD:SOT-23
- removed R2, R4, R7: 10k, Resistor_SMD:R_0603_1608Metric
- removed R3, R5, R8: 1k, Resistor_SMD:R_0603_1608Metric
- moved R16 2.49 mm to (127.8, 125.5), turned to 0 degrees
Connections:
- J1 pad 2: /X_OC -> /X_MASSO
- J3 pad 2: /Y_OC -> /Y_MASSO
- J5 pad 2: /Z_OC -> /Z_MASSO
- R1 pad 2: VDD -> /X_MASSO
- R6 pad 2: VDD -> /Y_MASSO
- R9 pad 2: VDD -> /Z_MASSO
- U1 pad 9: unconnected-(U1-GND-Pad9) -> GND
Routing:
- net VDD: track 198.9 -> 0.00 mm
- net +5V: track 71.6 -> 0.00 mm, vias 2 -> 0
- net /X_MASSO: track 69.3 -> 0.00 mm
- net /Y_MASSO: track 59.6 -> 0.00 mm
- net /TOUCH_OUT: track 56.6 -> 0.00 mm
- net /SPINDLE_STOP: track 45.6 -> 0.00 mm, vias 1 -> 0
- net /LASER_EN: track 37.2 -> 0.00 mm
- net GND: track 35.1 -> 0.00 mm, vias 1 -> 0
- net /LASER_ON_OC: track 32.7 -> 0.00 mm
- net /Z_MASSO: track 31.6 -> 0.00 mm
- net /SPINDLE_STOP_OC: track 30.9 -> 0.00 mm
- net /Y_OC: track 22.6 -> 0.00 mm
- net /Z_OC: track 12.7 -> 0.00 mm
- net Net-(D2-A): track 11.9 -> 0.00 mm
- net /X_OC: track 10.6 -> 0.00 mm
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