File: pulsegen/pulsegen.kicad_pcb (KiCad board)
At the start: 2 copper layers, 160 x 61 mm, 30 parts, among them J1 Screw_Terminal_01x01, J2 Screw_Terminal_01x01, J3 Screw_Terminal_01x01, J4 Screw_Terminal_01x01, Q1 QM6006D, Q3 QM6015D, Q4 QM6006D, Q5 QM6015D, SW1 SW_Push, SW3 RotaryEncoder_Switch, U2 MCP6001R, U3 LM7805_TO220, U4 ATmega328-A

Commit message: Typos and reord
Parts:
- added C1: 10u, Resistor_SMD:R_1206_3216Metric, F.Cu at (154.1, 106.3)
- added C2: C, Resistor_SMD:R_0603_1608Metric, F.Cu at (158.9, 105.9)
- added C3: 10u, Resistor_SMD:R_1206_3216Metric, F.Cu at (154.1, 109.6)
- added C4: 10u, Resistor_SMD:R_1206_3216Metric, F.Cu at (154.1, 112.9)
- added H1: MountingHole, MountingHole:MountingHole_3.2mm_M3, F.Cu at (80.1, 124.9)
- added H2: MountingHole, MountingHole:MountingHole_3.2mm_M3, F.Cu at (204.5, 76.5)
- added H4: MountingHole, MountingHole:MountingHole_3.2mm_M3, F.Cu at (77.5, 75.5)
- added H5: MountingHole, MountingHole:MountingHole_3.2mm_M3, F.Cu at (221.4, 123.9)
Routing:
- net GND: track 0.00 -> 248.2 mm
- net VCC: track 0.00 -> 131.6 mm, vias 0 -> 1
- net VDD: track 0.00 -> 116.8 mm
- net Net-(U4-PB0): track 0.00 -> 107.8 mm
- net Ismooth: track 0.00 -> 89.2 mm
- net Net-(U4-PD2): track 0.00 -> 86.7 mm
- net Net-(U4-PB1): track 0.00 -> 83.3 mm, vias 0 -> 2
- net Net-(U4-PD6): track 0.00 -> 64.6 mm, vias 0 -> 2
- net Net-(U2--): track 0.00 -> 64.1 mm
- net Net-(U4-PB2): track 0.00 -> 59.8 mm, vias 0 -> 2
- net Net-(U4-PD3): track 0.00 -> 58.9 mm, vias 0 -> 1
- net Net-(U4-PD4): track 0.00 -> 57.3 mm, vias 0 -> 1
- net Net-(U4-PD0): track 0.00 -> 53.0 mm, vias 0 -> 1
- net Net-(Q1-S): track 0.00 -> 48.8 mm
- net Net-(J1-Pin_1): track 0.00 -> 46.3 mm, vias 0 -> 1
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Other:
- outline, holes or cut-outs redrawn
