File: pulsegen/pulsegen.kicad_sch (KiCad schematic)
At the start: 35 parts, among them J1 Screw_Terminal_01x01, J2 Screw_Terminal_01x01, J3 Screw_Terminal_01x01, J4 Screw_Terminal_01x01, J5 AVR-ISP-6, Q1 QM6006D, Q3 QM6015D, Q4 QM6006D, Q5 QM6015D, SW1 SW_Push, SW3 RotaryEncoder_Switch, U2 MCP6001R, U3 LM7805_TO220, U4 ATmega328-A

Commit message: Typos and reord
Parts:
- added H1, H2, H4, H5: MountingHole, MountingHole:MountingHole_3.2mm_M3, symbol Mechanical:MountingHole
- C1, C3, C4: footprint (none) -> Resistor_SMD:R_1206_3216Metric
- C2: footprint (none) -> Resistor_SMD:R_0603_1608Metric
