File: cnc/central_control/modbus.kicad_sch (KiCad schematic)
At the start: 5 parts, among them J1 3pins, J4 DE9_Receptacle, U5 LT1785AxS8

Commit message: On-going
Parts:
- removed C3: 100n, Capacitor_SMD:C_0603_1608Metric_Pad1.08x0.95mm_HandSolder, symbol Device:C
- removed J1: 3pins, Connector_Phoenix_MC:PhoenixContact_MCV_1,5_3-G-3.81_1x03_P3.81mm_Vertical, symbol Connector:Screw_Terminal_01x03
- removed J4: DE9_Receptacle, Connector_Dsub:DSUB-9_Female_Vertical_P2.77x2.84mm_MountingHoles, symbol Connector:DE9_Receptacle
- removed R26: 100K, Resistor_SMD:R_1206_3216Metric_Pad1.30x1.75mm_HandSolder, symbol Device:R
- removed U5: LT1785AxS8, Package_SO:SOIC-8_3.9x4.9mm_P1.27mm, symbol Interface_UART:LT1785AxS8
