File: cnc/central_control/central_control.kicad_pcb (KiCad board)
At the start: 2 copper layers, 103 x 107 mm, 145 parts, among them J1 Outputs, J10 GND, J11 3pins, J12 3pins, J13 3pins, J14 Modbus, J15 DE9_Receptacle, J16 Supply, J2 Outputs, J20 AVR-UPDI, J3 Inputs, J4 Inputs, J5 7pins, J6 3pins, J7 3pins, J8 Phoenix, J9 GND, U1 LMR33630ADDA, U10 PC817, U11 PCA9555PW, U12 PCA9555PW, U13 PCA9555PW, U14 PC817, U15 PC817, U16 PC817, U17 PC817, U18 PC817, U19 PC817, U2 LT1785AxS8, U3 ATtiny3226, U5 PC817, U6 PC817, U7 PC817, U8 PC817, U9 PC817

Commit message: Added 4 layers
Parts:
- removed J15: DE9_Receptacle, Connector_Dsub:DSUB-9_Socket_Vertical_P2.77x2.84mm_MountingHoles
- removed RN1: 10k, Resistor_THT:R_Array_SIP5
- added C11: 1nF 250V, Capacitor_SMD:C_0603_1608Metric_Pad1.08x0.95mm_HandSolder, F.Cu at (170.8, 60.7)
- added C15: 1nF 250V, Capacitor_SMD:C_0603_1608Metric_Pad1.08x0.95mm_HandSolder, F.Cu at (143.0, 87.0)
- added C16: 1nF 250V, Capacitor_SMD:C_0603_1608Metric_Pad1.08x0.95mm_HandSolder, F.Cu at (194.9, 60.5)
- added C17: 1nF 250V, Capacitor_SMD:C_0603_1608Metric_Pad1.08x0.95mm_HandSolder, F.Cu at (185.0, 60.7)
- added C18: 1nF 250V, Capacitor_SMD:C_0603_1608Metric_Pad1.08x0.95mm_HandSolder, F.Cu at (161.9, 60.7)
- added C19: 1nF 250V, Capacitor_SMD:C_0603_1608Metric_Pad1.08x0.95mm_HandSolder, F.Cu at (165.9, 60.7)
- added C20: 1nF 250V, Capacitor_SMD:C_0603_1608Metric_Pad1.08x0.95mm_HandSolder, F.Cu at (156.6, 73.4)
- added C21: 1nF 250V, Capacitor_SMD:C_0603_1608Metric_Pad1.08x0.95mm_HandSolder, F.Cu at (161.6, 73.4)
- added C22: 1nF 250V, Capacitor_SMD:C_0603_1608Metric_Pad1.08x0.95mm_HandSolder, F.Cu at (177.2, 60.7)
- added C23: 1nF 250V, Capacitor_SMD:C_0603_1608Metric_Pad1.08x0.95mm_HandSolder, F.Cu at (181.0, 60.7)
- added C24: 1nF 250V, Capacitor_SMD:C_0603_1608Metric_Pad1.08x0.95mm_HandSolder, F.Cu at (174.4, 73.2)
- added C25: 1nF 250V, Capacitor_SMD:C_0603_1608Metric_Pad1.08x0.95mm_HandSolder, F.Cu at (136.2, 73.9)
- added H1: MountingHole_Pad, MountingHole:MountingHole_3.2mm_M3_DIN965_Pad_TopBottom, F.Cu at (194.0, 76.0)
- added H2: MountingHole_Pad, MountingHole:MountingHole_3.2mm_M3_DIN965_Pad_TopBottom, F.Cu at (116.0, 65.0)
- added H3: MountingHole_Pad, MountingHole:MountingHole_3.2mm_M3_DIN965_Pad_TopBottom, F.Cu at (187.0, 140.0)
- added H4: MountingHole_Pad, MountingHole:MountingHole_3.2mm_M3_DIN965_Pad_TopBottom, F.Cu at (116.0, 140.0)
- added J17: DE9_Socket_MountingHoles, Connector_Dsub:DSUB-9_Pins_Vertical_P2.77x2.84mm_MountingHoles, F.Cu at (192.6, 105.0)
- added R82: 10K, Resistor_SMD:R_1206_3216Metric_Pad1.30x1.75mm_HandSolder, F.Cu at (142.2, 71.9)
- added R83: 10k, Resistor_SMD:R_1206_3216Metric_Pad1.30x1.75mm_HandSolder, F.Cu at (182.1, 73.2)
- added R84: 10K, Resistor_SMD:R_1206_3216Metric_Pad1.30x1.75mm_HandSolder, F.Cu at (130.8, 72.6)
- added R85: 10K, Resistor_SMD:R_1206_3216Metric_Pad1.30x1.75mm_HandSolder, F.Cu at (135.6, 71.4)
- J1, J2: value Outputs -> 6pins
- J10, J9: value GND -> Phoenix
- J13: value 3pins -> Screw_Terminal_01x01; footprint Connector_Phoenix_MC:PhoenixContact_MCV_1,5_3-G-3.81_1x03_P3.81mm_Vertical -> adarwoo:GroundPlot
- J14: value Modbus -> 3pins
- J16: value Supply -> Phoenix
- J3: value Inputs -> 6pins
- J4: value Inputs -> 7pins
- moved R4 56.0 mm to (179.8, 122.0), turned to 90 degrees
- moved R79 50.2 mm to (170.8, 87.5)
- moved U5 50.2 mm to (170.8, 83.8)
- moved U12 43.4 mm to (116.8, 74.9)
- moved TP1 36.9 mm to (161.0, 117.0)
- moved R26 36.1 mm to (140.3, 87.5)
- moved U7 36.1 mm to (140.3, 83.8)
- moved R6 36.0 mm to (138.8, 125.3)
- moved R5 36.0 mm to (138.8, 128.9)
- moved R77 35.0 mm to (160.7, 87.5)
- moved U16 35.0 mm to (160.7, 83.8)
- moved U13 33.8 mm to (136.6, 136.5), turned to 90 degrees
- moved D1 25.9 mm to (167.5, 118.0)
- moved R76 24.8 mm to (155.6, 87.5)
- moved U17 24.8 mm to (155.6, 83.8)
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Connections:
- C1 pad 2: Earth -> GND
- C10 pad 2: Earth -> GND
- C12 pad 2: Earth -> GND
- C13 pad 2: Earth -> GND
- C14 pad 2: Earth -> GND
- C2 pad 2: Earth -> GND
- C3 pad 2: Earth -> GND
- C5 pad 2: Earth -> GND
- C6 pad 2: Earth -> GND
- C7 pad 1: Earth -> GND
- C8 pad 1: Earth -> GND
- C9 pad 2: Earth -> GND
- D10 pad 1: Earth -> GND
- D11 pad 1: Earth -> GND
- D12 pad 1: Earth -> GND
- D13 pad 1: Earth -> GND
- D14 pad 1: Earth -> GND
- D15 pad 1: Earth -> GND
- D16 pad 1: Earth -> GND
- D17 pad 1: Earth -> GND
- D18 pad 1: Earth -> GND
- D2 pad 1: Earth -> GND
- D3 pad 1: Earth -> GND
- D4 pad 1: Earth -> GND
- D5 pad 1: Earth -> GND
- D6 pad 1: Earth -> GND
- D7 pad 1: Earth -> GND
- D8 pad 1: Earth -> GND
- D9 pad 1: Earth -> GND
- J10 pad 1: Earth -> GND
- J10 pad 2: Earth -> GND
- J12 pad 1: Earth -> GND
- J12 pad 2: Earth -> GND
- J12 pad 3: Earth -> GND
- J13 pad 1: RS- -> GND
- J14 pad 3: Earth -> GND
- J16 pad 2: Earth -> GND
- J20 pad 6: Earth -> GND
- J6 pad 3: Earth -> GND
- J7 pad 3: Earth -> GND
- J8 pad 2: Earth -> GND
- J9 pad 1: Earth -> GND
- J9 pad 2: Earth -> GND
- R2 pad 1: Earth -> GND
- R3 pad 1: Earth -> GND
- R4 pad 1: Earth -> GND
- R44 pad 1: /Connections/MSO_IN0 -> CYCLE_START
- R45 pad 1: /Connections/MSO_IN1 -> HOME_MACHINE
- R46 pad 1: /Connections/MSO_IN2 -> CYCLE_STOP
- R47 pad 1: /Connections/MSO_IN3 -> GOTO_HOME
- R48 pad 1: /Connections/MSO_IN4 -> GOTO_PARK
- R49 pad 1: /Connections/MSO_IN5 -> OPEN_CHUCK
- R50 pad 1: /Connections/MSO_IN6 -> DOOR_OPEN_CLOSE
- R51 pad 1: /Connections/MSO_IN7 -> AUTOLOAD_GCODE_1
- R52 pad 1: /Connections/MSO_IN8 -> AUTOLOAD_GCODE_2
- R53 pad 1: /Connections/MSO_IN9 -> AUTOLOAD_GCODE_3
- R54 pad 1: /Connections/MSO_IN10 -> DOOR_SENSOR_INPUT
- R55 pad 1: /Connections/MSO_IN11 -> AIR_PRESSURE_LOW
- R60 pad 1: /Connections/MSO_OUT_TO_IN_1 -> TOWER_RED
- R61 pad 1: unconnected-(R61-Pad1) -> TOWER_YELLOW
- R62 pad 1: unconnected-(R62-Pad1) -> TOWER_GREEN
- R63 pad 1: unconnected-(R63-Pad1) -> DOOR_OPEN_CLOSE
- R64 pad 1: unconnected-(R64-Pad1) -> TOOL_AIR_BLAST_CLEANING
- R65 pad 1: unconnected-(R65-Pad1) -> CHUCK_PRESSURE
- R66 pad 1: unconnected-(R66-Pad1) -> Net-(J4-Pin_1)
- R66 pad 2: Net-(J4-Pin_1) -> SPARE_INPUT
- R67 pad 1: unconnected-(R67-Pad1) -> TOUCH_SCREEN_BEEP
- R68 pad 1: unconnected-(R68-Pad1) -> SOUNDER
- R69 pad 1: unconnected-(R69-Pad1) -> LIGHT_ON_OFF
- R70 pad 1: unconnected-(R70-Pad1) -> LASER_CROSSHAIR
- R71 pad 1: unconnected-(R71-Pad1) -> CAMERA_LIGHT
- R72 pad 1: unconnected-(R72-Pad1) -> ~{ES}
- TP2 pad 1: Earth -> GND
- U1 pad 1: Earth -> GND
- U1 pad 9: Earth -> GND
- U11 pad 12: Earth -> GND
- U11 pad 21: Earth -> GND
- U11 pad 3: Earth -> GND
- U12 pad 10: unconnected-(U12-IO0_6-Pad10) -> DOOR_OPEN_CLOSE
- U12 pad 12: Earth -> GND
- U12 pad 16: unconnected-(U12-IO1_3-Pad16) -> AIR_PRESSURE_LOW
- U12 pad 17: unconnected-(U12-IO1_4-Pad17) -> DOOR_SENSOR_INPUT
- U12 pad 18: unconnected-(U12-IO1_5-Pad18) -> AUTOLOAD_GCODE_3
- U12 pad 19: unconnected-(U12-IO1_6-Pad19) -> AUTOLOAD_GCODE_2
- U12 pad 2: Earth -> GND
- U12 pad 20: unconnected-(U12-IO1_7-Pad20) -> AUTOLOAD_GCODE_1
- U12 pad 21: Earth -> GND
- U12 pad 3: Earth -> GND
- U12 pad 4: /I2C/MSO_OUT0 -> CYCLE_START
- U12 pad 5: /I2C/MSO_OUT1 -> HOME_MACHINE
- U12 pad 6: /I2C/MSO_OUT2 -> CYCLE_STOP
- U12 pad 7: unconnected-(U12-IO0_3-Pad7) -> GOTO_HOME
- U12 pad 8: unconnected-(U12-IO0_4-Pad8) -> GOTO_PARK
- U12 pad 9: unconnected-(U12-IO0_5-Pad9) -> OPEN_CHUCK
- U13 pad 10: /I2C/MSO_IN6 -> unconnected-(U13-IO0_6-Pad10)
- U13 pad 11: /I2C/MSO_IN7 -> SPARE_INPUT
- U13 pad 12: Earth -> GND
- U13 pad 13: /I2C/MSO_IN8 -> TOUCH_SCREEN_BEEP
- U13 pad 14: /I2C/MSO_IN9 -> SOUNDER
- U13 pad 15: /I2C/MSO_IN10 -> LIGHT_ON_OFF
- U13 pad 16: /I2C/MSO_IN11 -> LASER_CROSSHAIR
- U13 pad 17: /I2C/MSO_IN12 -> CAMERA_LIGHT
- U13 pad 18: /I2C/MSO_IN13 -> ~{ES}
- U13 pad 19: /I2C/MSO_IN14 -> unconnected-(U13-IO1_6-Pad19)
- U13 pad 2: Earth -> GND
- U13 pad 20: /I2C/MSO_IN15 -> unconnected-(U13-IO1_7-Pad20)
- U13 pad 21: Earth -> GND
- U13 pad 3: Earth -> GND
- U13 pad 4: /I2C/MSO_IN0 -> TOWER_RED
- U13 pad 5: /I2C/MSO_IN1 -> TOWER_YELLOW
- U13 pad 6: /I2C/MSO_IN2 -> TOWER_GREEN
- U13 pad 7: /I2C/MSO_IN3 -> DOOR_OPEN_CLOSE
- U13 pad 8: /I2C/MSO_IN4 -> TOOL_AIR_BLAST_CLEANING
- U13 pad 9: /I2C/MSO_IN5 -> CHUCK_PRESSURE
- U14 pad 2: Earth -> GND
- U14 pad 3: Earth -> GND
- U15 pad 2: Earth -> GND
- U15 pad 3: Earth -> GND
- U16 pad 2: Earth -> GND
- U16 pad 3: Earth -> GND
- U17 pad 2: Earth -> GND
- U17 pad 3: Earth -> GND
- U18 pad 2: Earth -> GND
- U18 pad 3: Earth -> GND
- U19 pad 2: Earth -> GND
- U19 pad 3: Earth -> GND
- U2 pad 5: Earth -> GND
- U3 pad 20: Earth -> GND
- U5 pad 2: Earth -> GND
- U5 pad 3: Earth -> GND
- U6 pad 2: Earth -> GND
- U6 pad 3: Earth -> GND
Routing:
- net OC_IN_DOOR_IS_UP: track 0.00 -> 73.8 mm
- net OC_IN_DOOR_IS_CLOSED: track 0.00 -> 72.2 mm
- net +24V: track 0.00 -> 57.7 mm
- net GND: track 0.00 -> 54.2 mm, vias 0 -> 4
- net DOOR_OPEN_CLOSE: track 0.00 -> 54.2 mm
- net CHUCK_PRESSURE: track 0.00 -> 47.8 mm
- net Net-(U11-IO0_1): track 0.00 -> 33.8 mm
- net TOOL_AIR_BLAST_CLEANING: track 0.00 -> 33.6 mm
- net OC_IN_SPINDLE_IS_ON: track 0.00 -> 33.3 mm
- net OC_OUT_LIGHT: track 0.00 -> 32.8 mm
- net Net-(U11-IO0_2): track 0.00 -> 30.3 mm
- net AIR_PRESSURE_LOW: track 0.00 -> 27.8 mm
- net Net-(U11-IO0_3): track 0.00 -> 27.1 mm
- net SPARE_INPUT: track 0.00 -> 25.5 mm
- net DOOR_SENSOR_INPUT: track 0.00 -> 25.2 mm
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- added copper zone on In2.Cu, net +24V
- added copper zone on In1.Cu, net GND
- added copper zone on In2.Cu, net VCC
Other:
- copper layers 2 -> 4

Commit message: Diff pair in place
Parts:
- moved U2 21.7 mm to (175.5, 140.0)
Routing:
- net RS-: track 0.00 -> 67.6 mm
- net RS+: track 0.00 -> 66.5 mm

Commit message: Sent to production
Parts:
- removed C15, C21: 1nF 250V, Capacitor_SMD:C_0603_1608Metric_Pad1.08x0.95mm_HandSolder
- removed R10, R18, R19, R7, R8, R9: 332, Resistor_SMD:R_1206_3216Metric_Pad1.30x1.75mm_HandSolder
- removed R26: 3k32, Resistor_SMD:R_1206_3216Metric_Pad1.30x1.75mm_HandSolder
- removed R77: 560, Resistor_SMD:R_1206_3216Metric_Pad1.30x1.75mm_HandSolder
- removed R82: 10K, Resistor_SMD:R_1206_3216Metric_Pad1.30x1.75mm_HandSolder
- removed U16, U7: PC817, Package_DIP:DIP-4_W7.62mm
- added F1: ~, adarwoo:Murata_NFM61R, F.Cu at (186.3, 107.5)
- added F2: ~, adarwoo:Murata_NFM61R, F.Cu at (182.1, 92.8)
- C11, C16, C17, C18, C19, C20, C22, C23, C24, C25: footprint Capacitor_SMD:C_0603_1608Metric_Pad1.08x0.95mm_HandSolder -> Capacitor_SMD:C_1206_3216Metric_Pad1.33x1.80mm_HandSolder
- J13: value Screw_Terminal_01x01 -> ~
- R16: value 332 -> 10K
- R27, R28, R29: value 3k32 -> 2k21
- moved R12 65.2 mm to (213.5, 134.7)
- moved R22 52.1 mm to (181.8, 127.1), turned to 0 degrees
- moved R21 51.8 mm to (181.8, 123.7), turned to 0 degrees
- moved R13 45.9 mm to (175.7, 121.3), turned to -90 degrees
- moved C14 39.5 mm to (141.9, 66.0), turned to -90 degrees
- moved TP1 38.8 mm to (199.8, 116.7)
- moved G*** 35.2 mm to (162.8, 93.9)
- moved R20 32.0 mm to (184.0, 115.2), turned to -90 degrees
- moved C10 30.4 mm to (152.8, 103.2), turned to 90 degrees
- moved R28 30.1 mm to (154.5, 81.9)
- moved U14 30.0 mm to (164.7, 77.9)
- moved U9 30.0 mm to (154.5, 77.9)
- moved U10 30.0 mm to (159.6, 77.9)
- moved R81 30.0 mm to (164.7, 81.9)
- moved R29 30.0 mm to (159.6, 81.9)
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Connections:
- net Net-(C5-Pad1) renamed /Power supply/RAW_VCC
- J17 pad 0: unconnected-(J17-PAD-Pad0) -> GND
- J5 pad 4: OC_OUT_LIGHT -> OC_OUT_LASER_CROSS
- J5 pad 5: OC_OUT_LASER_CROSS -> OC_OUT_CAMERA_LIGHT
- J5 pad 6: OC_OUT_CAMERA_LIGHT -> OC_OUT_RELEASE_STEPPERS
- J5 pad 7: OC_OUT_RELEASE_STEPPERS -> OC_OUT_ES
- R16 pad 1: Net-(U3-PB2) -> IO_INT
- R16 pad 2: ISO_IN_SPARE_0 -> VCC
- R17 pad 1: Net-(U3-PB3) -> Net-(U3-PA5)
- R17 pad 2: ISO_IN_SPINDLE_IS_ON -> IO_INT
- R50 pad 1: DOOR_OPEN_CLOSE -> OPEN_CLOSE_DOOR
- R66 pad 2: SPARE_INPUT -> TOUCH_SCREEN_BEEP
- R67 pad 1: TOUCH_SCREEN_BEEP -> SOUNDER
- R68 pad 1: SOUNDER -> LASER_CROSSHAIR
- R69 pad 1: LIGHT_ON_OFF -> CAMERA_LIGHT
- R70 pad 1: LASER_CROSSHAIR -> SPARE_INPUT_1
- R71 pad 1: CAMERA_LIGHT -> SPARE_INPUT_2
- R79 pad 1: ISO_OUT_SPARE_0 -> ISO_OUT_CAMERA_LIGHT
- U11 pad 2: VCC -> GND
- U11 pad 21: GND -> VCC
- U12 pad 1: IO_INT -> unconnected-(U12-~{INT}-Pad1)
- U12 pad 10: DOOR_OPEN_CLOSE -> OPEN_CLOSE_DOOR
- U13 pad 10: unconnected-(U13-IO0_6-Pad10) -> TOUCH_SCREEN_BEEP
- U13 pad 11: SPARE_INPUT -> SOUNDER
- U13 pad 13: TOUCH_SCREEN_BEEP -> LASER_CROSSHAIR
- U13 pad 14: SOUNDER -> CAMERA_LIGHT
- U13 pad 15: LIGHT_ON_OFF -> SPARE_INPUT_1
- U13 pad 16: LASER_CROSSHAIR -> SPARE_INPUT_2
- U13 pad 17: CAMERA_LIGHT -> ~{ES}
- U13 pad 18: ~{ES} -> ISO_IN_SPINDLE_IS_ON
- U13 pad 19: unconnected-(U13-IO1_6-Pad19) -> ISO_IN_DOOR_IS_DOWN
- U13 pad 2: GND -> VCC
- U13 pad 20: unconnected-(U13-IO1_7-Pad20) -> ISO_IN_DOOR_IS_UP
- U13 pad 3: GND -> VCC
- U3 pad 12: Net-(U3-PC0) -> ISO_OUT_RELEASE_STEPPERS
- U3 pad 13: Net-(U3-PC1) -> ISO_OUT_LASER_CROSS
- U3 pad 14: Net-(U3-PC2) -> ISO_OUT_CAMERA_LIGHT
- U3 pad 15: Net-(U3-PC3) -> unconnected-(U3-PC3-Pad15)
- U3 pad 3: unconnected-(U3-PA5-Pad3) -> Net-(U3-PA5)
- U3 pad 6: Net-(U3-PB5) -> ISO_OUT_TOWER_LIGHT_GREEN
- U3 pad 7: Net-(U3-PB4) -> ISO_OUT_TOWER_LIGHT_YELLOW
- U3 pad 8: Net-(U3-PB3) -> ISO_OUT_TOWER_LIGHT_RED
- U3 pad 9: Net-(U3-PB2) -> ISO_OUT_ES
Routing:
- net VCC: track 9.05 -> 139.9 mm, vias 2 -> 20
- net ISO_IN_SPINDLE_IS_ON: track 3.10 -> 94.6 mm, vias 0 -> 1
- net SDA: track 0.00 -> 83.3 mm, vias 0 -> 2
- net ISO_IN_DOOR_IS_DOWN: track 2.34 -> 74.0 mm
- net SCL: track 18.0 -> 86.6 mm
- net ISO_IN_DOOR_IS_UP: track 4.01 -> 67.1 mm
- net ISO_OUT_RELEASE_STEPPERS: track 0.00 -> 58.1 mm
- net Net-(U3-PA2): track 4.54 -> 58.8 mm, vias 0 -> 2
- net ISO_OUT_TOWER_LIGHT_GREEN: track 0.00 -> 51.0 mm
- net UPDI: track 2.41 -> 52.1 mm
- net OC_OUT_ES: track 2.34 -> 51.1 mm
- net ISO_OUT_TOWER_LIGHT_YELLOW: track 0.00 -> 47.9 mm
- net ISO_OUT_CAMERA_LIGHT: track 0.00 -> 47.2 mm
- net ISO_OUT_LASER_CROSS: track 0.00 -> 45.6 mm
- net ISO_OUT_TOWER_LIGHT_RED: track 0.00 -> 45.3 mm
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- added copper zone on B.Cu, net +24V
- added copper zone on F.Cu, net +24V
- added copper zone on F.Cu, net /Power supply/RAW_VCC
- added copper zone on B.Cu, net GND
- added copper zone on F.Cu, net GND
- added copper zone on F.Cu, net Net-(U1-SW)
- added copper zone on F.Cu, net VCC
- added copper zone on F.Cu, net VDD
Other:
- board text added: "1"
- board text added: "2"
- board text added: "3"
- board text added: "4"
- board text added: "4/25"
- board text added: "CNC1.2 Ctrl Rev.B"
- board text removed: "CNC1.2 Ctrl Rev.A"
