File: cnc/central_control/i2c.kicad_sch (KiCad schematic)
At the start: 38 parts, among them U2 PCA9555PW, U3 PCA9555PW, U4 PCA9555PW

Commit message: On-going
Parts:
- removed D16, D8: LED, LED_THT:LED_D3.0mm, symbol Device:LED
- removed R27, R8: 432, Resistor_SMD:R_1206_3216Metric_Pad1.30x1.75mm_HandSolder, symbol Device:R
- D5: renamed from D1; value LED -> GRN
- renumbered C5 to C12, C2 to C13, C4 to C14, D6 to D10, D7 to D11, D9 to D12, D10 to D13, D11 to D14, D12 to D15, D13 to D16, D14 to D17, D15 to D18, D2 to D6, D3 to D7, D4 to D8, D5 to D9, R1 to R30, R2 to R31, R3 to R32, R4 to R33, R5 to R34, R6 to R35, R7 to R36, R11 to R37, R12 to R38, R14 to R39, R15 to R40, R16 to R41, R17 to R42, R25 to R43, U4 to U11, U3 to U12, U2 to U13
Connections:
- net MSO_OUT0: now reaches U12.4 (IO0_0)
- net MSO_OUT1: now reaches U12.5 (IO0_1)
- net MSO_OUT2: now reaches U12.6 (IO0_2)
Other:
- note removed: "| D# | Color | Function | Detail | |----|--------|---------------------------|------------------------------------------------------------------------| | 1 | Green | OC Door Openning | | | 2 | Green | OC Door Closing | | | 3 | Green | OC Spindle is on | | | 4 | Green | OC In spare | | | 5 | Yellow | OC Out release steppers | | | 6 | Yellow | OC out spare 0 | | | 7 | Yellow | Open collectors outp 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"
- moved on the sheet: C12, C13, C14, D5, R30, R31, R32, R33, R34, R35, R36, R37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

Commit message: Sent to production
Parts:
- added R16: 10K, Resistor_SMD:R_1206_3216Metric_Pad1.30x1.75mm_HandSolder, symbol Device:R
Connections:
- net GND: now also U11.2 (A1); no longer U11.21 (A0), U13.2 (A1), U13.3 (A2)
- net IO_INT: now also R16.1; no longer U12.1 (~{INT})
- net VCC: now also U11.21 (A0), U13.2 (A1), U13.3 (A2), R16.2; no longer U11.2 (A1)
- net OPEN_CLOSE_DOOR: now reaches U12.10 (IO0_6)
- net AIR_PRESSURE_LOW: now reaches U12.16 (IO1_3)
- net DOOR_SENSOR_INPUT: now reaches U12.17 (IO1_4)
- net AUTOLOAD_GCODE_3: now reaches U12.18 (IO1_5)
- net AUTOLOAD_GCODE_2: now reaches U12.19 (IO1_6)
- net AUTOLOAD_GCODE_1: now reaches U12.20 (IO1_7)
- net GOTO_HOME: now reaches U12.7 (IO0_3)
- net GOTO_PARK: now reaches U12.8 (IO0_4)
- net OPEN_CHUCK: now reaches U12.9 (IO0_5)
- net MSO_IN0 renamed TOWER_RED
- net MSO_IN1 renamed TOWER_YELLOW
- net MSO_IN10 renamed SPARE_INPUT_1
- net MSO_IN11 renamed SPARE_INPUT_2
- net MSO_IN12 renamed ~{ES}
- net MSO_IN13 renamed ISO_IN_SPINDLE_IS_ON
- net MSO_IN14 renamed ISO_IN_DOOR_IS_DOWN
- net MSO_IN15 renamed ISO_IN_DOOR_IS_UP
- net MSO_IN2 renamed TOWER_GREEN
- net MSO_IN3 renamed DOOR_OPEN_CLOSE
- net MSO_IN4 renamed TOOL_AIR_BLAST_CLEANING
- net MSO_IN5 renamed CHUCK_PRESSURE
- net MSO_IN6 renamed TOUCH_SCREEN_BEEP
- net MSO_IN7 renamed SOUNDER
- net MSO_IN8 renamed LASER_CROSSHAIR
- net MSO_IN9 renamed CAMERA_LIGHT
- net MSO_OUT0 renamed CYCLE_START
- net MSO_OUT1 renamed HOME_MACHINE
- net MSO_OUT2 renamed CYCLE_STOP
Other:
- note added: "I^{2}C Address = 0x20"
- note added: "I^{2}C Address = 0x21"
- note added: "I^{2}C Address = 0x26"
