File: cnc/central_control/isolated.kicad_sch (KiCad schematic)
At the start: 14 parts, among them U16 PC817, U17 PC817, U18 PC817, U19 PC817, U20 PC817, U21 PC817, U22 PC817, U7 PC817

Commit message: On-going
Parts:
- removed RN3: 3k31, Resistor_THT:R_Array_SIP5, symbol Device:R_Network04
- removed U16, U7: PC817, Package_DIP:DIP-4_W7.62mm, symbol Isolator:PC817
- added R24, R25: 3k32, Resistor_SMD:R_1206_3216Metric_Pad1.30x1.75mm_HandSolder, symbol Device:R
- renumbered R92 to R26, R93 to R27, R94 to R28, R95 to R29, U22 to U10, U17 to U5, U18 to U6, U19 to U7, U20 to U8, U21 to U9
Connections:
- net ISO_OUT_SPARE_2 is gone; now on net ISO_OUT_SPARE_0: U5.1
- net OC_OUT_SPARE_2 is gone; now on net OC_OUT_SPARE_0: U5.4
- net GND: now also R24.1, R25.1
- net at U5.2: now also R25.2
- net at U6.2: now also R24.2

Commit message: From scratch
Parts:
- removed R24, R25: 3k32, Resistor_SMD:R_1206_3216Metric_Pad1.30x1.75mm_HandSolder, symbol Device:R
- added R74, R75, R76, R77, R78, R79, R80, R81: 560, Resistor_SMD:R_1206_3216Metric_Pad1.30x1.75mm_HandSolder, symbol Device:R
- added U14, U15, U16, U17, U18, U19: PC817, Package_DIP:DIP-4_W7.62mm, symbol Isolator:PC817
Connections:
- net GND: now also U5.2, U6.2, U14.2, U14.3, U15.2, U15.3, U16.2, U16.3, U17.2, U17.3, U18.2, U18.3, U19.2, U19.3
- net ISO_OUT_RELEASE_STEPPERS: now also R80.1; no longer U6.1
- net ISO_OUT_SPARE_0: now also R79.1; no longer U5.1
- net OC_OUT_SPARE_0 renamed OC_OUT_CAMERA_LIGHT
- new net: R75.2, U18.1
- new net: R79.2, U5.1
- new net: R74.2, U19.1
- new net: R77.2, U16.1
- new net: R81.2, U14.1
- new net: R76.2, U17.1
- new net: R78.2, U15.1
- new net: R80.2, U6.1
- new net ISO_OUT_ES: R81.1
- new net ISO_OUT_LASER_CROSS: R78.1
- new net ISO_OUT_LIGHT: R77.1
- new net ISO_OUT_TOWER_LIGHT_GREEN: R76.1
- new net ISO_OUT_TOWER_LIGHT_RED: R74.1
- new net ISO_OUT_TOWER_LIGHT_YELLOW: R75.1
- new net OC_OUT_ES: U14.4
- new net OC_OUT_LASER_CROSS: U15.4
- new net OC_OUT_LIGHT: U16.4
- new net OC_OUT_TOWER_LIGHT_GREEN: U17.4
- new net OC_OUT_TOWER_LIGHT_RED: U19.4
- new net OC_OUT_TOWER_LIGHT_YELLOW: U18.4
Other:
- moved on the sheet: R26, R27, R28, R29, RN1, U10, U5, U6, U7, U8, U9

Commit message: Sent to production
Parts:
- removed R26: 3k32, Resistor_SMD:R_1206_3216Metric_Pad1.30x1.75mm_HandSolder, symbol Device:R
- removed R77: 560, Resistor_SMD:R_1206_3216Metric_Pad1.30x1.75mm_HandSolder, symbol Device:R
- removed RN1: 10k, Resistor_THT:R_Array_SIP5, symbol Device:R_Network04
- removed U16, U7: PC817, Package_DIP:DIP-4_W7.62mm, symbol Isolator:PC817
- added C11, C16, C17, C18, C19, C20, C22, C23, C24, C25: 1nF 250V, Capacitor_SMD:C_1206_3216Metric_Pad1.33x1.80mm_HandSolder, symbol Device:C
- added R83: 10k, Resistor_SMD:R_1206_3216Metric_Pad1.30x1.75mm_HandSolder, symbol Device:R
- added R84, R85: 10K, Resistor_SMD:R_1206_3216Metric_Pad1.30x1.75mm_HandSolder, symbol Device:R
- R27, R28, R29: value 3k32 -> 2k21
Connections:
- net GND: now also C11.2, C16.2, C17.2, C18.2, C19.2, C20.2, C22.2, C23.2, C24.2, C25.2, R83.2, R84.2, R85.2
- net ISO_IN_DOOR_IS_DOWN: now also R85.1
- net ISO_IN_DOOR_IS_UP: now also R84.1
- net ISO_IN_SPINDLE_IS_ON: now also R83.1
- net OC_IN_DOOR_IS_CLOSED: now also C11.1
- net OC_IN_DOOR_IS_UP: now also C17.1
- net OC_IN_SPINDLE_IS_ON: now also C16.1
- net OC_OUT_CAMERA_LIGHT: now also C23.1
- net OC_OUT_ES: now also C25.1
- net OC_OUT_LASER_CROSS: now also C22.1
- net OC_OUT_RELEASE_STEPPERS: now also C24.1
- net OC_OUT_TOWER_LIGHT_GREEN: now also C20.1
- net OC_OUT_TOWER_LIGHT_RED: now also C18.1
- net OC_OUT_TOWER_LIGHT_YELLOW: now also C19.1
- net ISO_OUT_SPARE_0 renamed ISO_OUT_CAMERA_LIGHT
Other:
- moved on the sheet: R27, R28, R29, R74, R75, R76, U10, U17, U18, U19, U8, U9
