File: cnc/central_control/power.kicad_sch (KiCad schematic)
At the start: 17 parts, among them U15 LMR33630ADDA

Commit message: On-going
Parts:
- renumbered C14 to C1, C15 to C2, C16 to C3, C17 to C4, C18 to C5, C19 to C6, C20 to C7, D20 to D1, F3 to F1, F4 to F2, L2 to L1, R75 to R1, R76 to R2, R77 to R3, TP4 to TP1, TP3 to TP2, U15 to U1
Changed lines of the file:
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@@
 (kicad_sch
-	(version 20231120)
+	(version 20250114)
 	(generator "eeschema")
-	(generator_version "8.0")
+	(generator_version "9.0")
 	(paper "A4")
 	(junction
@@
 		(on_board yes)
 		(dnp no)
-		(property "Reference" "D20"
+		(property "Reference" "D1"
 			(at 245.872 92.456 0)
 			(effects
@@
 			(project "central_control"
 				(path "/24bc57b9-acf8-493e-9df6-7015f7e1bb8a/8bb737e4-ae38-4c12-905d-9a7f99a5ad7b"
-					(reference "D20")
+					(reference "D1")
 					(unit 1)
 				)
@@
 		(on_board yes)
 		(dnp no)
-		(property "Reference" "C16"
+		(property "Reference" "C3"
 			(at 127 101.5999 0)
 			(effects
@@
 			(project "central_control"
 				(path "/24bc57b9-acf8-493e-9df6-7015f7e1bb8a/8bb737e4-ae38-4c12-905d-9a7f99a5ad7b"
-					(reference "C16")
+					(reference "C3")
 					(unit 1)
 				)
@@
 		(on_board yes)
 		(dnp no)
-		(property "Reference" "R75"
+		(property "Reference" "R1"
 			(at 177.8 89.916 90)
 			(effects
@@
 			(project "central_control"
 				(path "/24bc57b9-acf8-493e-9df6-7015f7e1bb8a/8bb737e4-ae38-4c12-905d-9a7f99a5ad7b"
-					(reference "R75")
+					(reference "R1")
 					(unit 1)
 				)
@@
 		(dnp no)
 		(fields_autoplaced yes)
-		(property "Reference" "F4"
+		(property "Reference" "F2"
 			(at 190.5 80.01 0)
 			(effects
@@
 			(project "central_control"
 				(path "/24bc57b9-acf8-493e-9df6-7015f7e1bb8a/8bb737e4-ae38-4c12-905d-9a7f99a5ad7b"
-					(reference "F4")
+					(reference "F2")
 					(unit 1)
 				)
@@
 		(on_board yes)
 		(dnp no)
-		(property "Reference" "C18"
+		(property "Reference" "C5"
 			(at 166.878 103.124 0)
 			(effects
@@
 			(project "central_control"
 				(path "/24bc57b9-acf8-493e-9df6-7015f7e1bb8a/8bb737e4-ae38-4c12-905d-9a7f99a5ad7b"
-					(reference "C18")
+					(reference "C5")
 					(unit 1)
 				)
@@
 		(on_board yes)
 		(dnp no)
-		(property "Reference" "TP4"
+		(property "Reference" "TP1"
 			(at 201.168 48.768 0)
 			(effects
@@
 			(project "central_control"
 				(path "/24bc57b9-acf8-493e-9df6-7015f7e1bb8a/8bb737e4-ae38-4c12-905d-9a7f99a5ad7b"
-					(reference "TP4")
+					(reference "TP1")
 					(unit 1)
 				)
@@
 		(on_board yes)
 		(dnp no)
-		(property "Reference" "R77"
+		(property "Reference" "R3"
 			(at 245.11 102.87 90)
 			(effects
@@
 			(project "central_control"
 				(path "/24bc57b9-acf8-493e-9df6-7015f7e1bb8a/8bb737e4-ae38-4c12-905d-9a7f99a5ad7b"
-					(reference "R77")
+					(reference "R3")
 					(unit 1)
 				)
@@
 		(dnp no)
 		(fields_autoplaced yes)
-		(property "Reference" "#PWR053"
+		(property "Reference" "#PWR04"
 			(at 196.85 52.07 0)
 			(effects
@@
 			(project "central_control"
 				(path "/24bc57b9-acf8-493e-9df6-7015f7e1bb8a/8bb737e4-ae38-4c12-905d-9a7f99a5ad7b"
-					(reference "#PWR053")
+					(reference "#PWR04")
 					(unit 1)
 				)
@@
 		(on_board yes)
 		(dnp no)
-		(property "Reference" "C20"
+		(property "Reference" "C7"
 			(at 212.09 100.076 0)
 			(effects
@@
 			(project "central_control"
 				(path "/24bc57b9-acf8-493e-9df6-7015f7e1bb8a/8bb737e4-ae38-4c12-905d-9a7f99a5ad7b"
-					(reference "C20")
+					(reference "C7")
 					(unit 1)
 				)
@@
 		(dnp no)
 		(fields_autoplaced yes)
-		(property "Reference" "#PWR054"
+		(property "Reference" "#PWR05"
 			(at 209.55 60.96 0)
 			(effects
@@
 			(project "central_control"
 				(path "/24bc57b9-acf8-493e-9df6-7015f7e1bb8a/8bb737e4-ae38-4c12-905d-9a7f99a5ad7b"
-					(reference "#PWR054")
+					(reference "#PWR05")
 					(unit 1)
 				)
@@
 		(on_board yes)
 		(dnp no)
-		(property "Reference" "C14"
+		(property "Reference" "C1"
 			(at 105.918 99.314 0)
 			(effects
@@
 			(project "central_control"
 				(path "/24bc57b9-acf8-493e-9df6-7015f7e1bb8a/8bb737e4-ae38-4c12-905d-9a7f99a5ad7b"
-					(reference "C14")
+					(reference "C1")
 					(unit 1)
 				)
@@
 		(dnp no)
 		(fields_autoplaced yes)
-		(property "Reference" "U15"
+		(property "Reference" "U1"
 			(at 137.16 77.47 0)
 			(effects
@@
 			(project "central_control"
 				(path "/24bc57b9-acf8-493e-9df6-7015f7e1bb8a/8bb737e4-ae38-4c12-905d-9a7f99a5ad7b"
-					(reference "U15")
+					(reference "U1")
 					(unit 1)
 				)
@@
 		(dnp no)
 		(fields_autoplaced yes)
-		(property "Reference" "#PWR052"
+		(property "Reference" "#PWR08"
 			(at 242.57 115.57 0)
 			(effects
@@
 			(project "central_control"
 				(path "/24bc57b9-acf8-493e-9df6-7015f7e1bb8a/8bb737e4-ae38-4c12-905d-9a7f99a5ad7b"
-					(reference "#PWR052")
+					(reference "#PWR08")
 					(unit 1)
 				)
@@
 		(dnp no)
 		(fields_autoplaced yes)
-		(property "Reference" "TP3"
+		(property "Reference" "TP2"
 			(at 212.09 50.0379 0)
 			(effects
@@
 			(project "central_control"
 				(path "/24bc57b9-acf8-493e-9df6-7015f7e1bb8a/8bb737e4-ae38-4c12-905d-9a7f99a5ad7b"
-					(reference "TP3")
+					(reference "TP2")
 					(unit 1)
 				)
@@
 		(dnp no)
 		(fields_autoplaced yes)
-		(property "Reference" "#PWR047"
+		(property "Reference" "#PWR03"
 			(at 149.86 129.54 0)
 			(effects
@@
 			(project "central_control"
 				(path "/24bc57b9-acf8-493e-9df6-7015f7e1bb8a/8bb737e4-ae38-4c12-905d-9a7f99a5ad7b"
-					(reference "#PWR047")
+					(reference "#PWR03")
 					(unit 1)
 				)
@@
 		(dnp no)
 		(fields_autoplaced yes)
-		(property "Reference" "#PWR051"
+		(property "Reference" "#PWR06"
 			(at 210.82 83.82 0)
 			(effects
@@
 			(project "central_control"
 				(path "/24bc57b9-acf8-493e-9df6-7015f7e1bb8a/8bb737e4-ae38-4c12-905d-9a7f99a5ad7b"
-					(reference "#PWR051")
+					(reference "#PWR06")
 					(unit 1)
 				)
@@
 		(dnp no)
 		(fields_autoplaced yes)
-		(property "Reference" "#PWR044"
+		(property "Reference" "#PWR01"
 			(at 86.36 83.82 0)
 			(effects
@@
 			(project "central_control"
 				(path "/24bc57b9-acf8-493e-9df6-7015f7e1bb8a/8bb737e4-ae38-4c12-905d-9a7f99a5ad7b"
-					(reference "#PWR044")
+					(reference "#PWR01")
 					(unit 1)
 				)
@@
 		(dnp no)
 		(fields_autoplaced yes)
-		(property "Reference" "C17"
+		(property "Reference" "C4"
 			(at 153.67 77.47 90)
 			(effects
@@
 			(project "central_control"
 				(path "/24bc57b9-acf8-493e-9df6-7015f7e1bb8a/8bb737e4-ae38-4c12-905d-9a7f99a5ad7b"
-					(reference "C17")
+					(reference "C4")
 					(unit 1)
 				)
@@
 		(on_board yes)
 		(dnp no)
-		(property "Reference" "C15"
+		(property "Reference" "C2"
 			(at 112.522 94.234 0)
 			(effects
@@
 			(project "central_control"
 				(path "/24bc57b9-acf8-493e-9df6-7015f7e1bb8a/8bb737e4-ae38-4c12-905d-9a7f99a5ad7b"
-					(reference "C15")
+					(reference "C2")
 					(unit 1)
 				)
@@
 		(dnp no)
 		(fields_autoplaced yes)
-		(property "Reference" "F3"
+		(property "Reference" "F1"
 			(at 99.06 80.01 0)
 			(effects
@@
 			(project "central_control"
 				(path "/24bc57b9-acf8-493e-9df6-7015f7e1bb8a/8bb737e4-ae38-4c12-905d-9a7f99a5ad7b"
-					(reference "F3")
+					(reference "F1")
 					(unit 1)
 				)
@@
 		(dnp no)
 		(fields_autoplaced yes)
-		(property "Reference" "L2"
+		(property "Reference" "L1"
 			(at 165.1 80.01 90)
 			(effects
@@
 			(project "central_control"
 				(path "/24bc57b9-acf8-493e-9df6-7015f7e1bb8a/8bb737e4-ae38-4c12-905d-9a7f99a5ad7b"
-					(reference "L2")
+					(reference "L1")
 					(unit 1)
 				)
@@
 		(on_board yes)
 		(dnp no)
-		(property "Reference" "C19"
+		(property "Reference" "C6"
 			(at 203.962 100.584 0)
 			(effects
@@
 			(project "central_control"
 				(path "/24bc57b9-acf8-493e-9df6-7015f7e1bb8a/8bb737e4-ae38-4c12-905d-9a7f99a5ad7b"
-					(reference "C19")
+					(reference "C6")
 					(unit 1)
 				)
@@
 		(dnp no)
 		(fields_autoplaced yes)
-		(property "Reference" "#PWR048"
+		(property "Reference" "#PWR07"
 			(at 242.57 90.17 0)
 			(effects
@@
 			(project "central_control"
 				(path "/24bc57b9-acf8-493e-9df6-7015f7e1bb8a/8bb737e4-ae38-4c12-905d-9a7f99a5ad7b"
-					(reference "#PWR048")
+					(reference "#PWR07")
 					(unit 1)
 				)
@@
 		(on_board yes)
 		(dnp no)
-		(property "Reference" "R76"
+		(property "Reference" "R2"
 			(at 177.8 105.156 90)
 			(effects
@@
 			(project "central_control"
 				(path "/24bc57b9-acf8-493e-9df6-7015f7e1bb8a/8bb737e4-ae38-4c12-905d-9a7f99a5ad7b"
-					(reference "R76")
+					(reference "R2")
 					(unit 1)
 				)
@@
 		(dnp no)
 		(fields_autoplaced yes)
-		(property "Reference" "#PWR050"
+		(property "Reference" "#PWR02"
 			(at 113.03 83.82 0)
 			(effects
@@
 			(project ""
 				(path "/24bc57b9-acf8-493e-9df6-7015f7e1bb8a/8bb737e4-ae38-4c12-905d-9a7f99a5ad7b"
-					(reference "#PWR050")
-					(unit 1)
-				)
+					(reference "#PWR02")
+					(unit 1)
+				)

Commit message: Sent to production
Parts:
- removed F1, F2: ~, Adarwoo:Murata_NFM61R, symbol ARex:NFM611R30
- added F1, F2: ~, Adarwoo:Murata_NFM61R, symbol Arex:NFM611R30
Connections:
- net +24V: now also F1.1
- net GND: now also F1.2, F2.2
- net VCC: now also F2.3
- net VDD: now also F1.3
- net RAW_VCC: now reaches C5.1, L1.2, R1.2
- net RAW_VCC: now also F2.1
