File: cnc/central_control/micro.kicad_sch (KiCad schematic)
At the start: 26 parts, among them J2 AVR-UPDI, U1 ATtiny3226

Commit message: On-going
Parts:
- removed R23: 332, Resistor_SMD:R_0805_2012Metric_Pad1.20x1.40mm_HandSolder, symbol Device:R
- removed R73: 332, Resistor_SMD:R_1206_3216Metric_Pad1.30x1.75mm_HandSolder, symbol Device:R
- added C8: 100n, Capacitor_SMD:C_0603_1608Metric_Pad1.08x0.95mm_HandSolder, symbol Device:C
- added R12: 332, Resistor_SMD:R_1206_3216Metric_Pad1.30x1.75mm_HandSolder, symbol Device:R
- added R4: 100K, Resistor_SMD:R_1206_3216Metric_Pad1.30x1.75mm_HandSolder, symbol Device:R
- added TP3: IDLE, TestPoint:TestPoint_Loop_D3.50mm_Drill0.9mm_Beaded, symbol Connector:TestPoint
- added U2: LT1785AxS8, Package_SO:SOIC-8_3.9x4.9mm_P1.27mm, symbol Interface_UART:LT1785AxS8
- R10: renamed from R20; footprint Resistor_SMD:R_0805_2012Metric_Pad1.20x1.40mm_HandSolder -> Resistor_SMD:R_1206_3216Metric_Pad1.30x1.75mm_HandSolder
- R14: renamed from R29; footprint Resistor_SMD:R_0805_2012Metric_Pad1.20x1.40mm_HandSolder -> Resistor_SMD:R_1206_3216Metric_Pad1.30x1.75mm_HandSolder
- R15: renamed from R28; footprint Resistor_SMD:R_0805_2012Metric_Pad1.20x1.40mm_HandSolder -> Resistor_SMD:R_1206_3216Metric_Pad1.30x1.75mm_HandSolder
- R17: renamed from R24; footprint Resistor_SMD:R_0805_2012Metric_Pad1.20x1.40mm_HandSolder -> Resistor_SMD:R_1206_3216Metric_Pad1.30x1.75mm_HandSolder
- R18: renamed from R42; footprint Resistor_SMD:R_0805_2012Metric_Pad1.20x1.40mm_HandSolder -> Resistor_SMD:R_1206_3216Metric_Pad1.30x1.75mm_HandSolder
- R19: renamed from R72; footprint Resistor_SMD:R_0805_2012Metric_Pad1.20x1.40mm_HandSolder -> Resistor_SMD:R_1206_3216Metric_Pad1.30x1.75mm_HandSolder
- R7: renamed from R13; footprint Resistor_SMD:R_0805_2012Metric_Pad1.20x1.40mm_HandSolder -> Resistor_SMD:R_1206_3216Metric_Pad1.30x1.75mm_HandSolder
- R8: renamed from R18; footprint Resistor_SMD:R_0805_2012Metric_Pad1.20x1.40mm_HandSolder -> Resistor_SMD:R_1206_3216Metric_Pad1.30x1.75mm_HandSolder
- R9: renamed from R19; footprint Resistor_SMD:R_0805_2012Metric_Pad1.20x1.40mm_HandSolder -> Resistor_SMD:R_1206_3216Metric_Pad1.30x1.75mm_HandSolder
- renumbered C1 to C10, C21 to C9, D19 to D2, D21 to D3, D23 to D4, J2 to J1, R78 to R11, R21 to R13, R79 to R16, R74 to R20, R22 to R21, R80 to R22, R9 to R5, R10 to R6, U1 to U3
Connections:
- net GND: now also C8.1, R4.1, U2.5 (GND)
- net RS_TX_PULSE: now also U3.4 (PA6); no longer U3.3 (PA5)
- net RTXD: now also U2.1 (RO), U2.4 (DI)
- net VCC: now also C8.2, U2.8 (VCC)
- net XDIR: now also R4.2, U2.2 (~{RE}), U2.3 (DE)
- net at U3.18 (PA2): now also R12.1
- net at R16.1: now also U3.9 (PB2); no longer U3.4 (PA6)
- net OC_IN_SPARE renamed ISO_IN_SPARE_0
- net OUT0 renamed ISO_OUT_SPARE_0
- net OUT1 renamed ISO_OUT_SPARE_1
- net OUT2 renamed ISO_OUT_SPARE_2
- net OUT3 renamed ISO_OUT_RELEASE_STEPPERS
- new net IDLE: R12.2, TP3.1
- new net RS+: U2.7 (B)
- new net RS-: U2.6 (A)
Other:
- note added: "RS485"
- moved on the sheet: R16, R5, R6

Commit message: From scratch
Parts:
- renumbered J1 to J20
Changed lines of the file:
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@@
 		(on_board yes)
 		(dnp no)
-		(property "Reference" "J1"
+		(property "Reference" "J20"
 			(at 38.862 151.892 0)
 			(effects
@@
 			(project "central_control"
 				(path "/24bc57b9-acf8-493e-9df6-7015f7e1bb8a/4d858077-b048-410a-a113-2658348ba3c3"
-					(reference "J1")
+					(reference "J20")
 					(unit 1)
 				)

Commit message: On-going
Parts:
- removed R10, R16, R18, R19, R7, R8, R9: 332, Resistor_SMD:R_1206_3216Metric_Pad1.30x1.75mm_HandSolder, symbol Device:R
Connections:
- net ISO_OUT_RELEASE_STEPPERS: now also U3.12 (PC0)
- net at R17.1: now also U3.3 (PA5); no longer U3.8 (PB3)
- net ISO_OUT_TOWER_LIGHT_GREEN: now reaches U3.6 (PB5)
- net ISO_OUT_ES: now reaches U3.9 (PB2)
- net ISO_OUT_CAMERA_LIGHT: now reaches U3.14 (PC2)
- net ISO_OUT_LASER_CROSS: now reaches U3.13 (PC1)
- net ISO_OUT_TOWER_LIGHT_YELLOW: now reaches U3.7 (PB4)
- net ISO_IN_SPINDLE_IS_ON renamed IO_INT
- new net ISO_OUT_TOWER_LIGHT_RED: U3.8 (PB3)
Other:
- moved on the sheet: R11, R12, R13, R14, R15
