File: cnc/central_control/connections.kicad_sch (KiCad schematic)
At the start: 37 parts, among them J10 7pins, J11 Phoenix, J3 6pins, J5 6pins, J6 Screw_Terminal_01x04, J7 6pins, J8 4pins, J9 Screw_Terminal_01x01

Commit message: On-going
Parts:
- removed J6: Screw_Terminal_01x04, Connector_Phoenix_MC:PhoenixContact_MCV_1,5_4-G-3.81_1x04_P3.81mm_Vertical, symbol Connector:Screw_Terminal_01x04
- removed J8: 4pins, Connector_Phoenix_MC:PhoenixContact_MCV_1,5_4-G-3.81_1x04_P3.81mm_Vertical, symbol Connector:Screw_Terminal_01x04
- removed R43, R44, R45, R46: 332, Resistor_SMD:R_0805_2012Metric_Pad1.20x1.40mm_HandSolder, symbol Device:R
- added J13, J20, J21, J23, J24: 3pins, Connector_Phoenix_MC:PhoenixContact_MCV_1,5_3-G-3.81_1x03_P3.81mm_Vertical, symbol Connector:Screw_Terminal_01x03
- added J14: DE9_Receptacle, Connector_Dsub:DSUB-9_Socket_Vertical_P2.77x2.84mm_MountingHoles, symbol Connector:DE9_Receptacle
- added J17, J18, J22: Phoenix, Connector_Phoenix_MC:PhoenixContact_MCV_1,5_2-G-3.81_1x02_P3.81mm_Vertical, symbol Connector:Screw_Terminal_01x02
- added J19: 7pins, Connector_Phoenix_MC:PhoenixContact_MCV_1,5_7-G-3.81_1x07_P3.81mm_Vertical, symbol Connector:Screw_Terminal_01x07
- added J2: Screw_Terminal_01x04, Connector_Phoenix_MC:PhoenixContact_MCV_1,5_4-G-3.81_1x04_P3.81mm_Vertical, symbol Connector:Screw_Terminal_01x04
- added R56, R57, R58, R59: 332, Resistor_SMD:R_1206_3216Metric_Pad1.30x1.75mm_HandSolder, symbol Device:R
- J10: renamed from J9; footprint TerminalBlock_Wuerth:Wuerth_REDCUBE-THR_WP-THRBU_74650173_THR -> adarwoo:GroundPlot
- R44: renamed from R30; footprint Resistor_SMD:R_0805_2012Metric_Pad1.20x1.40mm_HandSolder -> Resistor_SMD:R_1206_3216Metric_Pad1.30x1.75mm_HandSolder
- R45: renamed from R31; footprint Resistor_SMD:R_0805_2012Metric_Pad1.20x1.40mm_HandSolder -> Resistor_SMD:R_1206_3216Metric_Pad1.30x1.75mm_HandSolder
- R46: renamed from R32; footprint Resistor_SMD:R_0805_2012Metric_Pad1.20x1.40mm_HandSolder -> Resistor_SMD:R_1206_3216Metric_Pad1.30x1.75mm_HandSolder
- R47: renamed from R33; footprint Resistor_SMD:R_0805_2012Metric_Pad1.20x1.40mm_HandSolder -> Resistor_SMD:R_1206_3216Metric_Pad1.30x1.75mm_HandSolder
- R48: renamed from R34; footprint Resistor_SMD:R_0805_2012Metric_Pad1.20x1.40mm_HandSolder -> Resistor_SMD:R_1206_3216Metric_Pad1.30x1.75mm_HandSolder
- R49: renamed from R35; footprint Resistor_SMD:R_0805_2012Metric_Pad1.20x1.40mm_HandSolder -> Resistor_SMD:R_1206_3216Metric_Pad1.30x1.75mm_HandSolder
- R50: renamed from R36; footprint Resistor_SMD:R_0805_2012Metric_Pad1.20x1.40mm_HandSolder -> Resistor_SMD:R_1206_3216Metric_Pad1.30x1.75mm_HandSolder
- R51: renamed from R37; footprint Resistor_SMD:R_0805_2012Metric_Pad1.20x1.40mm_HandSolder -> Resistor_SMD:R_1206_3216Metric_Pad1.30x1.75mm_HandSolder
- R52: renamed from R38; footprint Resistor_SMD:R_0805_2012Metric_Pad1.20x1.40mm_HandSolder -> Resistor_SMD:R_1206_3216Metric_Pad1.30x1.75mm_HandSolder
- R53: renamed from R39; footprint Resistor_SMD:R_0805_2012Metric_Pad1.20x1.40mm_HandSolder -> Resistor_SMD:R_1206_3216Metric_Pad1.30x1.75mm_HandSolder
- R54: renamed from R40; footprint Resistor_SMD:R_0805_2012Metric_Pad1.20x1.40mm_HandSolder -> Resistor_SMD:R_1206_3216Metric_Pad1.30x1.75mm_HandSolder
- R55: renamed from R41; footprint Resistor_SMD:R_0805_2012Metric_Pad1.20x1.40mm_HandSolder -> Resistor_SMD:R_1206_3216Metric_Pad1.30x1.75mm_HandSolder
- R60: renamed from R47; footprint Resistor_SMD:R_0805_2012Metric_Pad1.20x1.40mm_HandSolder -> Resistor_SMD:R_1206_3216Metric_Pad1.30x1.75mm_HandSolder
- R61: renamed from R48; footprint Resistor_SMD:R_0805_2012Metric_Pad1.20x1.40mm_HandSolder -> Resistor_SMD:R_1206_3216Metric_Pad1.30x1.75mm_HandSolder
- R62: renamed from R49; footprint Resistor_SMD:R_0805_2012Metric_Pad1.20x1.40mm_HandSolder -> Resistor_SMD:R_1206_3216Metric_Pad1.30x1.75mm_HandSolder
- R63: renamed from R50; footprint Resistor_SMD:R_0805_2012Metric_Pad1.20x1.40mm_HandSolder -> Resistor_SMD:R_1206_3216Metric_Pad1.30x1.75mm_HandSolder
- R64: renamed from R51; footprint Resistor_SMD:R_0805_2012Metric_Pad1.20x1.40mm_HandSolder -> Resistor_SMD:R_1206_3216Metric_Pad1.30x1.75mm_HandSolder
- R65: renamed from R52; footprint Resistor_SMD:R_0805_2012Metric_Pad1.20x1.40mm_HandSolder -> Resistor_SMD:R_1206_3216Metric_Pad1.30x1.75mm_HandSolder
- R66: renamed from R53; footprint Resistor_SMD:R_0805_2012Metric_Pad1.20x1.40mm_HandSolder -> Resistor_SMD:R_1206_3216Metric_Pad1.30x1.75mm_HandSolder
- R67: renamed from R54; footprint Resistor_SMD:R_0805_2012Metric_Pad1.20x1.40mm_HandSolder -> Resistor_SMD:R_1206_3216Metric_Pad1.30x1.75mm_HandSolder
- R68: renamed from R55; footprint Resistor_SMD:R_0805_2012Metric_Pad1.20x1.40mm_HandSolder -> Resistor_SMD:R_1206_3216Metric_Pad1.30x1.75mm_HandSolder
- R69: renamed from R56; footprint Resistor_SMD:R_0805_2012Metric_Pad1.20x1.40mm_HandSolder -> Resistor_SMD:R_1206_3216Metric_Pad1.30x1.75mm_HandSolder
- R70: renamed from R57; footprint Resistor_SMD:R_0805_2012Metric_Pad1.20x1.40mm_HandSolder -> Resistor_SMD:R_1206_3216Metric_Pad1.30x1.75mm_HandSolder
- R71: renamed from R58; footprint Resistor_SMD:R_0805_2012Metric_Pad1.20x1.40mm_HandSolder -> Resistor_SMD:R_1206_3216Metric_Pad1.30x1.75mm_HandSolder
- R72: renamed from R59; footprint Resistor_SMD:R_0805_2012Metric_Pad1.20x1.40mm_HandSolder -> Resistor_SMD:R_1206_3216Metric_Pad1.30x1.75mm_HandSolder
- renumbered J7 to J11, J10 to J12, J11 to J6, J3 to J7, J5 to J8
Connections:
- net GND is gone; now on net Earth: J6.2 (Pin_2)
- net +24V: now also J14.2, J14.4, J23.1 (Pin_1), J23.2 (Pin_2), J23.3 (Pin_3)
- net Earth: now also J13.3 (Pin_3), J14.1, J14.6, J17.1 (Pin_1), J17.2 (Pin_2), J18.1 (Pin_1), J18.2 (Pin_2), J20.3 (Pin_3), J21.3 (Pin_3), J22.2 (Pin_2), J24.1 (Pin_1), J24.2 (Pin_2), J24.3 (Pin_3)
- net MSO_OUT0 renamed MSO_OUT_TO_IN_1
- net MSO_OUT1: no longer names the net of R61.1
- net MSO_OUT10: no longer names the net of R70.1
- net MSO_OUT11: no longer names the net of R71.1
- net MSO_OUT12: no longer names the net of R72.1
- net MSO_OUT2: no longer names the net of R62.1
- net MSO_OUT3: no longer names the net of R63.1
- net MSO_OUT4: no longer names the net of R64.1
- net MSO_OUT5: no longer names the net of R65.1
- net MSO_OUT6: no longer names the net of R66.1
- net MSO_OUT7: no longer names the net of R67.1
- net MSO_OUT8: no longer names the net of R68.1
- net MSO_OUT9: no longer names the net of R69.1
- new net OC_IN_DOOR_IS_CLOSED: J20.2 (Pin_2)
- new net OC_IN_DOOR_IS_UP: J21.2 (Pin_2)
- new net OC_IN_SPINDLE_IS_ON: J22.1 (Pin_1)
- new net OC_OUT_RELEASE_STEPPERS: J19.7 (Pin_7)
- new net OC_OUT_SPARE_0: J19.6 (Pin_6)
- new net RS+: J13.2 (Pin_2), J14.5
- new net RS-: J13.1 (Pin_1), J14.9
- new net VCC: J14.7, J14.8
Other:
- moved on the sheet: J11, J12, J8, R50, R51, R52, R53, R54, R55, R60, R61, R62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

Commit message: From scratch
Parts:
- removed J2: Screw_Terminal_01x04, Connector_Phoenix_MC:PhoenixContact_MCV_1,5_4-G-3.81_1x04_P3.81mm_Vertical, symbol Connector:Screw_Terminal_01x04
- removed R56, R57, R58, R59: 332, Resistor_SMD:R_1206_3216Metric_Pad1.30x1.75mm_HandSolder, symbol Device:R
- renumbered J7 to J1, J17 to J10, J23 to J11, J24 to J12, J10 to J13, J13 to J14, J14 to J15, J6 to J16, J8 to J2, J11 to J3, J12 to J4, J19 to J5, J20 to J6, J21 to J7, J22 to J8, J18 to J9
Connections:
- net +24V: now also J6.1 (Pin_1), J7.1 (Pin_1)
- net OC_OUT_TOWER_LIGHT_RED: now reaches J5.1 (Pin_1)
- net OC_OUT_TOWER_LIGHT_YELLOW: now reaches J5.2 (Pin_2)
- net OC_OUT_TOWER_LIGHT_GREEN: now reaches J5.3 (Pin_3)
- net OC_OUT_LIGHT: now reaches J5.4 (Pin_4)
- net OC_OUT_LASER_CROSS: now reaches J5.5 (Pin_5)
- net OC_OUT_SPARE_0 renamed OC_OUT_CAMERA_LIGHT
Other:
- moved on the sheet: J11, J12, J8

Commit message: Sent to production
Parts:
- removed J15: DE9_Receptacle, Connector_Dsub:DSUB-9_Socket_Vertical_P2.77x2.84mm_MountingHoles, symbol Connector:DE9_Receptacle
- added H1, H2, H3, H4: MountingHole_Pad, MountingHole:MountingHole_3.2mm_M3_DIN965_Pad_TopBottom, symbol Mechanical:MountingHole_Pad
- added J17: DE9_Socket_MountingHoles, Connector_Dsub:DSUB-9_Pins_Vertical_P2.77x2.84mm_MountingHoles, symbol Connector:DE9_Socket_MountingHoles
- J13: value Screw_Terminal_01x01 -> ~
Connections:
- net OC_OUT_LIGHT is gone; now on net OC_OUT_LASER_CROSS: J5.4 (Pin_4)
- net +24V: now also J17.2, J17.4
- net OC_OUT_CAMERA_LIGHT: now also J5.5 (Pin_5); no longer J5.6 (Pin_6)
- net OC_OUT_LASER_CROSS: no longer J5.5 (Pin_5)
- net OC_OUT_RELEASE_STEPPERS: now also J5.6 (Pin_6); no longer J5.7 (Pin_7)
- net RS+: now also J17.5
- net RS-: now also J17.9
- net VCC: now also J17.7, J17.8
- net CHUCK_PRESSURE: now reaches R65.1
- net ~{ES}: now reaches R72.1
- net TOOL_AIR_BLAST_CLEANING: now reaches R64.1
- net LASER_CROSSHAIR: now reaches R68.1
- net CAMERA_LIGHT: now reaches R69.1
- net SOUNDER: now reaches R67.1
- net SPARE_INPUT_2: now reaches R71.1
- net DOOR_OPEN_CLOSE: now reaches R63.1
- net TOWER_GREEN: now reaches R62.1
- net at R66.1: now also J4.1 (Pin_1)
- net TOUCH_SCREEN_BEEP: now reaches R66.2
- net TOUCH_SCREEN_BEEP: no longer J4.1 (Pin_1)
- net SPARE_INPUT_1: now reaches R70.1
- net TOWER_YELLOW: now reaches R61.1
- net Earth renamed GND
- net GND: now also H1.1, H2.1, H3.1, H4.1, J17.0 (PAD), J17.1, J17.6
- net MSO_IN0 renamed CYCLE_START
- net MSO_IN1 renamed HOME_MACHINE
- net MSO_IN10 renamed DOOR_SENSOR_INPUT
- net MSO_IN11 renamed AIR_PRESSURE_LOW
- net MSO_IN2 renamed CYCLE_STOP
- net MSO_IN3 renamed GOTO_HOME
- net MSO_IN4 renamed GOTO_PARK
- net MSO_IN5 renamed OPEN_CHUCK
- net MSO_IN6 renamed OPEN_CLOSE_DOOR
- net MSO_IN7 renamed AUTOLOAD_GCODE_1
- net MSO_IN8 renamed AUTOLOAD_GCODE_2
- net MSO_IN9 renamed AUTOLOAD_GCODE_3
- net MSO_OUT_TO_IN_1 renamed TOWER_RED
- new net OC_OUT_ES: J5.7 (Pin_7)
Other:
- note added: "CNC Center TTL output to Masso inputs"
- note added: "Masso outputs to CNC Center TTL inputs"
- moved on the sheet: J1, J10, J11, J12, J13, J14, J16, J2, J3, J4, J5, J6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

Commit message: Sent to production
Parts:
- R72: value 332 -> 221
Changed lines of the file:
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@@
 			)
 		)
-		(property "Value" "332"
+		(property "Value" "221"
 			(at 192.024 88.9 90)
 			(effects
